File: 32V_AC_DC.kicad_sch (KiCad schematic)
At the start: 30 parts, among them J1 Conn_01x02_Pin, Q1 NMOS_Substrate, U1 OB2269CP

Commit message: 2nd commit
Parts:
- removed C1: C_Polarized_US, symbol Device:C_Polarized_US
- removed D1: D, symbol Device:D
- added C10, C11, C2, C4, C5, C7: C, symbol Device:C
- added CON3: LED, symbol Connector:Conn_01x02_Pin
- added D2, D5: D, symbol Device:D
- added D4, D6: D_Zener_Dual_CommonCathode_AKA, symbol Device:D_Zener_Dual_CommonCathode_AKA
- added EC3, EC4, EC5, EC7, EC8: C_Polarized_US, symbol Device:C_Polarized_US
- added J2: Conn_01x07_Pin, symbol Connector:Conn_01x07_Pin
- added J3: Conn_01x04_Pin, symbol Connector:Conn_01x04_Pin
- added JP1: Jumper_2_Bridged, symbol Jumper:Jumper_2_Bridged
- added JP4, R45: 0Ohm, symbol Device:R_US
- added L1, L2, L3, L4: L, symbol Device:L
- added PC1, PC2: 1008, symbol Isolator:Optocoupler_DC_PhotoNPN_AKEC
- added Q2, Q3, U3: ESDA5V3L, Package_TO_SOT_SMD:SOT-23-3, symbol Power_Protection:ESDA5V3L
- added Q5: KS6210, Package_TO_SOT_SMD:TO-252-2, symbol Transistor_FET:IPD50R3K0CE
- added R10, R11 (x2), R12, R14, R15, R16, R17, R19, R2, R21, R22, R24, R25, R26, R28, R29, R30, R32, R35, R36, R38, R43, R44, R5, R6: R_US, symbol Device:R_US
- added R20: 0.02 Ohm, symbol Device:R_US
- added U2: DP358, Package_SO:MSOP-8_3x3mm_P0.65mm, symbol Amplifier_Operational:AD8606ARM
- added ZD1, ZD2, ZD3: D_Zener, symbol Device:D_Zener
- RT1: renamed from RA3; value R_Variable_US -> 10k
- renumbered C5 to C1, C3 to C12, C4 to C13, D3 to D1
Connections:
- net GND: now also U1.1 (GND), C2.1, EC3.2, JP1.2 (B), PC1.2, R10.1; no longer R8.1
- net at Q1.3 (S), R3.2, R34.1: now also R8.1
- net at C12.1, C13.1, D2.1 (+)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: now also L1.1, R5.1
- net at C12.2, C13.2, D1.2 (A)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: now also L1.2
- net at U1.2 (FB): now also C2.2, PC1.1
- net at U1.3 (VIN): now also R6.2
- net at U1.4 (RI): now also R10.2
- net at U1.7 (VDD): now also D2.1 (K), EC3.1
- net at RT1.1: now also R19.1, U3.1 (K), U3.2 (K), ZD1.2 (A)
- net at RT1.2: now also R16.2
- new net: D4.1 (A), D4.3 (A), L4.2, R11.1, R12.1, R36.1
- new net: C4.1, R11.2, R12.2, R36.2
- new net: C7.1, R22.2
- new net: C7.2, D6.2 (K), EC7.1, EC8.1, J3.1 (Pin_1), R17.1, ZD3.1 (K)
- new net: C10.2, D5.2 (A), PC1.3, R21.1, ZD2.1 (K)
- new net: PC1.4, R21.2, R32.1
- new net: D2.2 (A), R2.1
- new net: L2.1, R2.2
- new net: R24.1, R32.2, ZD1.1 (K)
- new net: R5.2, R6.1
- new net: D6.1 (A), D6.3 (A), L3.1, R22.1
- new net: Q3.2 (K), R29.1, R30.1
- new net: J2.3 (Pin_3), R29.2
- new net: D5.1 (K), R11.1, R15.1, U2.1
- new net: C5.1, R44.1, U2.2 (-)
- new net: C5.2, R15.2
- new net: J2.1 (Pin_1), R35.2
- new net: JP1.1 (A), L2.2
- new net: PC2.1, R35.1
- new net: JP4.2, PC2.2
- new net: PC2.4, R45.2
- new net: Q5.1 (G), R26.2, R38.2
- new net: Q5.3 (S), R20.2, R38.1
- new net: Q3.3 (A), R25.2
- new net: Q2.2 (K), R25.1, R28.2
- new net: R16.1, R43.2, R45.1, U2.3 (+)
- new net: Q2.1 (K), R28.1
- new net: Q2.3 (A), R26.1
- new net GND3: C10.1, C11.2, EC4.2, EC5.2, EC7.2, EC8.2, J2.2 (Pin_2), J2.4 (Pin_4), J2.5 (Pin_5), J3.2 (Pin_2), J3.3 (Pin_3), JP4.1, L3.2, L4.1, Q3.1 (K), R11.2, R14.2, R17.2, R20.1, R30.2, R43.1, R44.2, U3.3 (A), U3.4 (V-), ZD2.2 (A), ZD3.2 (A)
- new net GNDREF: PC2.3
- new net Vcc: R24.2, U3.8 (V+)
- new net Vout12V: C11.1, J2.6 (Pin_6), J2.7 (Pin_7), J3.4 (Pin_4)
- new net led+: C4.2, CON3.2 (Pin_2), D4.2 (K), EC4.1, EC5.1, R14.1, R19.2
- new net led-: CON3.1 (Pin_1), Q5.2 (D)
- no-connect marks 0 -> 1
Other:
- moved on the sheet: C1, C12, C13, C2, D1, D2, D7, EC1, EC2, F1, J1, Q1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
